File: Eagle files/TinyCard.brd (EAGLE design)
At the start: 86.4 x 55.9 mm, 35 parts, among them CN1 USBA_FEMALE, IC1 MAX619CSA, Q1 MOSFET-PCHANNELSMD, U5 SD_CARD_SOCKET4UCON

Commit message: Version 2 - 27th March 2025
Decoupling capacitors
Parts:
- added C6, C7: 1µF, microbuilder:_0805MP
Connections:
- net GND: now also C6.1, C7.1
- net POWER: now also C6.2, C7.2
Routing:
- net GND: track 182.4 -> 183.5 mm
- net POWER: track 79.3 -> 78.5 mm
Changed lines of the file:
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@@
 <setting verticaltext="up"/>
 </settings>
-<grid distance="0.05" unitdist="inch" unit="inch" style="lines" multiple="2" display="yes" altdistance="0.0125" altunitdist="inch" altunit="inch"/>
+<grid distance="0.05" unitdist="inch" unit="inch" style="lines" multiple="2" display="yes" altdistance="0.00625" altunitdist="inch" altunit="inch"/>
 <layers>
 <layer number="1" name="Top" color="4" fill="1" visible="yes" active="yes"/>
@@
 <attribute name="VALUE" x="74.2425" y="48.5125" size="0.4064" layer="28" rot="MR0"/>
 </element>
+<element name="C6" library="microbuilder" package="_0805MP" value="1µF" x="46.0375" y="23.1775" smashed="yes" rot="MR0">
+<attribute name="NAME" x="46.6725" y="23.97125" size="0.8128" layer="26" ratio="18" rot="MR0"/>
+<attribute name="VALUE" x="47.625" y="21.9075" size="0.4064" layer="28" ratio="10" rot="MR0"/>
+</element>
+<element name="C7" library="microbuilder" package="_0805MP" value="1µF" x="10.16" y="29.21" smashed="yes" rot="MR90">
+<attribute name="NAME" x="9.36625" y="29.845" size="0.8128" layer="26" ratio="18" rot="MR270"/>
+<attribute name="VALUE" x="8.89" y="27.6225" size="0.4064" layer="28" ratio="10" rot="MR90"/>
+</element>
 </elements>
 <signals>
@@
 <contactref element="CN2" pad="6"/>
 <wire x1="22.86" y1="27.94" x2="29.21" y2="21.59" width="0.8128" layer="16"/>
-<wire x1="29.21" y1="21.59" x2="35.8775" y2="21.59" width="0.8128" layer="16"/>
-<wire x1="35.8775" y1="21.59" x2="38.731128125" y2="21.555153125" width="0.8128" layer="16"/>
-<wire x1="38.731128125" y1="21.555153125" x2="46.993871875" y2="21.624846875" width="0.8128" layer="16"/>
-<wire x1="46.993871875" y1="21.624846875" x2="59.3725" y2="21.59" width="0.8128" layer="16"/>
 <wire x1="59.3725" y1="21.59" x2="63.2968" y2="25.4" width="0.8128" layer="16"/>
 <contactref element="U5" pad="6"/>
@@
 <wire x1="46.97" y1="28.4335" x2="46.97" y2="25.9875" width="0.8128" layer="16"/>
 <wire x1="46.97" y1="25.9875" x2="46.993871875" y2="25.9875" width="0.4064" layer="16"/>
-<wire x1="46.97" y1="25.9875" x2="46.97" y2="21.64871875" width="0.8128" layer="16"/>
-<wire x1="46.97" y1="21.64871875" x2="46.993871875" y2="21.624846875" width="0.4064" layer="16"/>
 <wire x1="71.755" y1="18.415" x2="71.755" y2="18.7325" width="0.4064" layer="16"/>
 <wire x1="71.755" y1="18.7325" x2="74.3025" y2="21.28" width="0.4064" layer="16"/>
@@
 <wire x1="71.7425" y1="49.2125" x2="71.7425" y2="48.5265" width="0.8128" layer="16"/>
 <wire x1="71.7425" y1="48.5265" x2="73.5965" y2="46.6725" width="0.8128" layer="16"/>
+<contactref element="C6" pad="1"/>
+<wire x1="46.97" y1="25.9875" x2="47.0535" y2="25.9875" width="0.8128" layer="16"/>
+<wire x1="47.0535" y1="25.9875" x2="47.0535" y2="23.1775" width="0.8128" layer="16"/>
+<wire x1="29.21" y1="21.59" x2="59.3725" y2="21.59" width="0.8128" layer="16"/>
+<contactref element="C7" pad="1"/>
+<wire x1="10.16" y1="28.194" x2="12.4968" y2="28.194" width="0.8128" layer="16"/>
+<wire x1="12.4968" y1="28.194" x2="12.4968" y2="27.94" width="0.8128" layer="16"/>
 </signal>
 <signal name="GND1" class="1">
@@
 </signal>
 <signal name="POWER">
-<wire x1="22.5425" y1="30.48" x2="29.845" y2="23.1775" width="0.4064" layer="16"/>
-<wire x1="29.845" y1="23.1775" x2="43.815" y2="23.1775" width="0.4064" layer="16"/>
-<wire x1="43.815" y1="23.1775" x2="56.8325" y2="23.1775" width="0.4064" layer="1"/>
-<wire x1="56.8325" y1="23.1775" x2="61.595" y2="27.94" width="0.4064" layer="1"/>
+<wire x1="22.5425" y1="30.48" x2="29.845" y2="23.1775" width="0.8128" layer="16"/>
+<wire x1="29.845" y1="23.1775" x2="43.72" y2="23.1775" width="0.8128" layer="16"/>
+<wire x1="56.8325" y1="23.1775" x2="61.595" y2="27.94" width="0.8128" layer="1"/>
 <contactref element="CN2" pad="4"/>
 <contactref element="U5" pad="4"/>
 <wire x1="43.72" y1="25.9875" x2="43.83" y2="25.9875" width="0.4064" layer="16"/>
 <wire x1="43.83" y1="25.9875" x2="43.83" y2="29.386" width="0.4064" layer="16"/>
-<wire x1="43.83" y1="29.386" x2="43.83" y2="23.1925" width="0.4064" layer="16"/>
-<wire x1="43.83" y1="23.1925" x2="43.815" y2="23.1775" width="0.4064" layer="16"/>
-<via x="43.815" y="23.1775" extent="1-16" drill="0.5"/>
+<wire x1="43.83" y1="23.1925" x2="43.72" y2="23.1775" width="0.4064" layer="16"/>
 <contactref element="Q1" pad="3"/>
 <contactref element="JP1" pad="2"/>
 <contactref element="R1" pad="2"/>
 <contactref element="JP4" pad="9"/>
-<wire x1="10.16" y1="33.274" x2="10.16" y2="31.75" width="0.4064" layer="16"/>
-<wire x1="10.16" y1="31.75" x2="11.43" y2="30.48" width="0.4064" layer="16"/>
-<wire x1="11.43" y1="30.48" x2="12.9032" y2="30.48" width="0.4064" layer="16"/>
-<wire x1="63.7032" y1="27.94" x2="67.6275" y2="27.94" width="0.4064" layer="16"/>
-<wire x1="71.6075" y1="30.48" x2="70.1675" y2="30.48" width="0.4064" layer="16"/>
-<wire x1="70.1675" y1="30.48" x2="67.6275" y2="27.94" width="0.4064" layer="16"/>
-<wire x1="61.595" y1="27.94" x2="63.7032" y2="27.94" width="0.4064" layer="1"/>
-<wire x1="22.5425" y1="30.48" x2="12.9032" y2="30.48" width="0.4064" layer="16"/>
+<wire x1="63.7032" y1="27.94" x2="67.6275" y2="27.94" width="0.8128" layer="16"/>
+<wire x1="71.6075" y1="30.48" x2="70.1675" y2="30.48" width="0.8128" layer="16"/>
+<wire x1="70.1675" y1="30.48" x2="67.6275" y2="27.94" width="0.8128" layer="16"/>
+<wire x1="61.595" y1="27.94" x2="63.7032" y2="27.94" width="0.8128" layer="1"/>
+<wire x1="22.5425" y1="30.48" x2="12.9032" y2="30.48" width="0.8128" layer="16"/>
+<contactref element="C6" pad="2"/>
+<wire x1="43.83" y1="23.1925" x2="43.72" y2="23.1925" width="0.8128" layer="16"/>
+<wire x1="43.72" y1="23.1925" x2="43.72" y2="25.9875" width="0.8128" layer="16"/>
+<wire x1="43.83" y1="23.1925" x2="45.0215" y2="23.1925" width="0.8128" layer="16"/>
+<wire x1="45.0215" y1="23.1925" x2="45.0215" y2="23.1775" width="0.8128" layer="16"/>
+<wire x1="56.8325" y1="23.1775" x2="43.72" y2="23.1775" width="0.8128" layer="1"/>
+<via x="43.72" y="23.1775" extent="1-16" drill="0.5"/>
+<wire x1="43.72" y1="23.1775" x2="43.72" y2="23.1925" width="0.8128" layer="16"/>
+<contactref element="C7" pad="2"/>
+<wire x1="10.16" y1="33.274" x2="10.16" y2="30.226" width="0.8128" layer="16"/>
+<wire x1="12.9032" y1="30.48" x2="10.16" y2="30.48" width="0.8128" layer="16"/>
+<wire x1="10.16" y1="30.48" x2="10.16" y2="30.226" width="0.8128" layer="16"/>
 </signal>
 <signal name="!ENABLE">
